File: neckmed/neckmed-3.sch (EAGLE design)
At the start: 9 parts, among them U1 HT7333, U2 GY-521MPU6050

Commit message: minus esp clearance
Connections:
- net GND: now also SW.2, U$1.GND@38; no longer SW.1, U1.GND
- net N$2: now also SW.1, U1.GND; no longer SW.2, U$1.GND@1
- net VCC: now also U$1.IO36
Other:
- moved on the sheet: SW
Changed lines of the file:
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@@
 <part name="P+3" library="supply1" library_urn="urn:adsk.eagle:library:371" deviceset="VCC" device=""/>
 <part name="CHARGER" library="B2B-XH-A" deviceset="B2B-XH-A" device=""/>
-<part name="GND4" library="supply1" library_urn="urn:adsk.eagle:library:371" deviceset="GND" device=""/>
 <part name="P+4" library="supply1" library_urn="urn:adsk.eagle:library:371" deviceset="VCC" device=""/>
 <part name="JP1" library="pinhead" library_urn="urn:adsk.eagle:library:325" deviceset="PINHD-1X2" device="" package3d_urn="urn:adsk.eagle:package:22435/2"/>
@@
 <part name="SUPPLY1" library="supply2" library_urn="urn:adsk.eagle:library:372" deviceset="GND" device=""/>
 <part name="P+5" library="supply1" library_urn="urn:adsk.eagle:library:371" deviceset="VCC" device=""/>
+<part name="P+6" library="supply1" library_urn="urn:adsk.eagle:library:371" deviceset="VCC" device=""/>
+<part name="SUPPLY2" library="supply2" library_urn="urn:adsk.eagle:library:372" deviceset="GND" device=""/>
 <part name="SW" library="B2B-XH-A" deviceset="B2B-XH-A" device=""/>
 </parts>
@@
 <attribute name="VALUE" x="-17.78" y="106.68" size="1.778" layer="96" rot="R180"/>
 </instance>
-<instance part="GND4" gate="1" x="12.7" y="73.66" smashed="yes">
-<attribute name="VALUE" x="10.16" y="71.12" size="1.778" layer="96"/>
-</instance>
 <instance part="P+4" gate="VCC" x="86.36" y="43.18" smashed="yes">
 <attribute name="VALUE" x="83.82" y="40.64" size="1.778" layer="96" rot="R90"/>
@@
 <attribute name="VALUE" x="5.08" y="58.42" size="1.778" layer="96" rot="R90"/>
 </instance>
-<instance part="SW" gate="G$1" x="17.78" y="86.36" smashed="yes" rot="R90">
-<attribute name="NAME" x="11.43" y="83.82" size="1.778" layer="95" rot="R90"/>
-<attribute name="VALUE" x="22.86" y="83.82" size="1.778" layer="96" rot="R90"/>
+<instance part="P+6" gate="VCC" x="22.86" y="60.96" smashed="yes" rot="R90">
+<attribute name="VALUE" x="25.4" y="58.42" size="1.778" layer="96" rot="R180"/>
+</instance>
+<instance part="SUPPLY2" gate="GND" x="71.12" y="68.58" smashed="yes" rot="R90">
+<attribute name="VALUE" x="74.295" y="66.675" size="1.778" layer="96" rot="R90"/>
+</instance>
+<instance part="SW" gate="G$1" x="45.72" y="93.98" smashed="yes">
+<attribute name="NAME" x="43.18" y="100.33" size="1.778" layer="95"/>
+<attribute name="VALUE" x="43.18" y="88.9" size="1.778" layer="96"/>
 </instance>
 </instances>
@@
 <pinref part="P+5" gate="VCC" pin="VCC"/>
 <pinref part="LED1" gate="G$1" pin="A"/>
+</segment>
+<segment>
+<pinref part="P+6" gate="VCC" pin="VCC"/>
+<pinref part="U$1" gate="G$1" pin="IO36"/>
 </segment>
 </net>
@@
 <junction x="68.58" y="91.44"/>
 <pinref part="CHARGER" gate="G$1" pin="1"/>
-<wire x1="38.1" y1="101.6" x2="38.1" y2="91.44" width="0.1524" layer="91"/>
 <junction x="38.1" y="91.44"/>
 <wire x1="2.54" y1="99.06" x2="2.54" y2="91.44" width="0.1524" layer="91"/>
@@
 <pinref part="C3" gate="G$1" pin="2"/>
 <pinref part="C1" gate="G$1" pin="2"/>
-<pinref part="U1" gate="G$1" pin="GND"/>
-<wire x1="38.1" y1="101.6" x2="53.34" y2="101.6" width="0.1524" layer="91"/>
-<wire x1="53.34" y1="101.6" x2="53.34" y2="106.68" width="0.1524" layer="91"/>
+<wire x1="38.1" y1="93.98" x2="38.1" y2="91.44" width="0.1524" layer="91"/>
+<pinref part="SW" gate="G$1" pin="2"/>
 </segment>
 <segment>
@@
 </segment>
 <segment>
-<pinref part="GND4" gate="1" pin="GND"/>
-<wire x1="15.24" y1="78.74" x2="12.7" y2="78.74" width="0.1524" layer="91"/>
-<wire x1="12.7" y1="78.74" x2="12.7" y2="76.2" width="0.1524" layer="91"/>
-<pinref part="SW" gate="G$1" pin="1"/>
-</segment>
-<segment>
 <pinref part="LED1" gate="G$1" pin="C"/>
 <pinref part="SUPPLY1" gate="GND" pin="GND"/>
+</segment>
+<segment>
+<pinref part="U$1" gate="G$1" pin="GND@38"/>
+<wire x1="63.5" y1="68.58" x2="68.58" y2="68.58" width="0.1524" layer="91"/>
+<pinref part="SUPPLY2" gate="GND" pin="GND"/>
+<wire x1="68.58" y1="68.58" x2="71.12" y2="68.58" width="0.1524" layer="91"/>
+<junction x="68.58" y="68.58"/>
 </segment>
 </net>
@@
 <net name="N$2" class="0">
 <segment>
-<pinref part="U$1" gate="G$1" pin="GND@1"/>
-<wire x1="25.4" y1="68.58" x2="20.32" y2="68.58" width="0.1524" layer="91"/>
-<wire x1="20.32" y1="68.58" x2="20.32" y2="78.74" width="0.1524" layer="91"/>
-<pinref part="SW" gate="G$1" pin="2"/>
-<wire x1="17.78" y1="78.74" x2="20.32" y2="78.74" width="0.1524" layer="91"/>
-</segment>
-</net>
+<pinref part="U1" gate="G$1" pin="GND"/>
+<wire x1="53.34" y1="101.6" x2="53.34" y2="106.68" width="0.1524" layer="91"/>
+<wire x1="38.1" y1="101.6" x2="53.34" y2="101.6" width="0.1524" layer="91"/>
+<wire x1="38.1" y1="101.6" x2="38.1" y2="96.52" width="0.1524" layer="91"/>
+<pinref part="SW" gate="G$1" pin="1"/>
+</segment>
+</net>

Commit message: move switch
Connections:
- net GND: now also SW.1, U1.GND; no longer CHARGER.1, LED1.C, SW.2
- net N$2: now also CHARGER.1, LED1.C, SW.2; no longer SW.1, U1.GND
Other:
- moved on the sheet: SW
Changed lines of the file:
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@@
 <part name="U1" library="HT7333" deviceset="HT7333" device=""/>
 <part name="LED1" library="led" library_urn="urn:adsk.eagle:library:259" deviceset="TLLR4400" device="" package3d_urn="urn:adsk.eagle:package:15797/1"/>
-<part name="SUPPLY1" library="supply2" library_urn="urn:adsk.eagle:library:372" deviceset="GND" device=""/>
 <part name="P+5" library="supply1" library_urn="urn:adsk.eagle:library:371" deviceset="VCC" device=""/>
 <part name="P+6" library="supply1" library_urn="urn:adsk.eagle:library:371" deviceset="VCC" device=""/>
@@
 <attribute name="VALUE" x="13.335" y="51.308" size="1.778" layer="96" rot="R90"/>
 </instance>
-<instance part="SUPPLY1" gate="GND" x="7.62" y="48.26" smashed="yes">
-<attribute name="VALUE" x="5.715" y="45.085" size="1.778" layer="96"/>
-</instance>
 <instance part="P+5" gate="VCC" x="7.62" y="60.96" smashed="yes">
 <attribute name="VALUE" x="5.08" y="58.42" size="1.778" layer="96" rot="R90"/>
@@
 <attribute name="VALUE" x="74.295" y="66.675" size="1.778" layer="96" rot="R90"/>
 </instance>
-<instance part="SW" gate="G$1" x="45.72" y="93.98" smashed="yes">
-<attribute name="NAME" x="43.18" y="100.33" size="1.778" layer="95"/>
-<attribute name="VALUE" x="43.18" y="88.9" size="1.778" layer="96"/>
+<instance part="SW" gate="G$1" x="-7.62" y="83.82" smashed="yes" rot="R270">
+<attribute name="NAME" x="-1.27" y="86.36" size="1.778" layer="95" rot="R270"/>
+<attribute name="VALUE" x="-12.7" y="86.36" size="1.778" layer="96" rot="R270"/>
 </instance>
 </instances>
@@
 <segment>
 <wire x1="68.58" y1="104.14" x2="68.58" y2="91.44" width="0.1524" layer="91"/>
-<wire x1="68.58" y1="91.44" x2="38.1" y2="91.44" width="0.1524" layer="91"/>
-<wire x1="38.1" y1="91.44" x2="17.78" y2="91.44" width="0.1524" layer="91"/>
+<wire x1="68.58" y1="91.44" x2="53.34" y2="91.44" width="0.1524" layer="91"/>
+<wire x1="53.34" y1="91.44" x2="17.78" y2="91.44" width="0.1524" layer="91"/>
 <wire x1="17.78" y1="91.44" x2="2.54" y2="91.44" width="0.1524" layer="91"/>
-<wire x1="2.54" y1="91.44" x2="-12.7" y2="91.44" width="0.1524" layer="91"/>
-<wire x1="-12.7" y1="91.44" x2="-12.7" y2="99.06" width="0.1524" layer="91"/>
 <wire x1="17.78" y1="101.6" x2="17.78" y2="91.44" width="0.1524" layer="91"/>
 <junction x="17.78" y="91.44"/>
 <pinref part="GND1" gate="1" pin="GND"/>
 <junction x="68.58" y="91.44"/>
-<pinref part="CHARGER" gate="G$1" pin="1"/>
-<junction x="38.1" y="91.44"/>
 <wire x1="2.54" y1="99.06" x2="2.54" y2="91.44" width="0.1524" layer="91"/>
 <junction x="2.54" y="91.44"/>
@@
 <pinref part="C3" gate="G$1" pin="2"/>
 <pinref part="C1" gate="G$1" pin="2"/>
-<wire x1="38.1" y1="93.98" x2="38.1" y2="91.44" width="0.1524" layer="91"/>
-<pinref part="SW" gate="G$1" pin="2"/>
+<pinref part="U1" gate="G$1" pin="GND"/>
+<wire x1="53.34" y1="106.68" x2="53.34" y2="91.44" width="0.1524" layer="91"/>
+<junction x="53.34" y="91.44"/>
+<pinref part="SW" gate="G$1" pin="1"/>
+<wire x1="2.54" y1="91.44" x2="-5.08" y2="91.44" width="0.1524" layer="91"/>
 </segment>
 <segment>
@@
 <pinref part="GND2" gate="1" pin="GND"/>
 <wire x1="78.74" y1="78.74" x2="78.74" y2="76.2" width="0.1524" layer="91"/>
-</segment>
-<segment>
-<pinref part="LED1" gate="G$1" pin="C"/>
-<pinref part="SUPPLY1" gate="GND" pin="GND"/>
 </segment>
 <segment>
@@
 <net name="N$2" class="0">
 <segment>
-<pinref part="U1" gate="G$1" pin="GND"/>
-<wire x1="53.34" y1="101.6" x2="53.34" y2="106.68" width="0.1524" layer="91"/>
-<wire x1="38.1" y1="101.6" x2="53.34" y2="101.6" width="0.1524" layer="91"/>
-<wire x1="38.1" y1="101.6" x2="38.1" y2="96.52" width="0.1524" layer="91"/>
-<pinref part="SW" gate="G$1" pin="1"/>
+<pinref part="CHARGER" gate="G$1" pin="1"/>
+<wire x1="-12.7" y1="91.44" x2="-12.7" y2="99.06" width="0.1524" layer="91"/>
+<wire x1="-7.62" y1="91.44" x2="-12.7" y2="91.44" width="0.1524" layer="91"/>
+<pinref part="SW" gate="G$1" pin="2"/>
+<wire x1="-12.7" y1="91.44" x2="-12.7" y2="48.26" width="0.1524" layer="91"/>
+<junction x="-12.7" y="91.44"/>
+<pinref part="LED1" gate="G$1" pin="C"/>
+<wire x1="7.62" y1="50.8" x2="5.08" y2="50.8" width="0.1524" layer="91"/>
+<wire x1="5.08" y1="50.8" x2="5.08" y2="48.26" width="0.1524" layer="91"/>
+<wire x1="-12.7" y1="48.26" x2="5.08" y2="48.26" width="0.1524" layer="91"/>
 </segment>
 </net>

Commit message: update xh library
Connections:
- net VCC: no longer U2.ADO
Changed lines of the file:
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@@
 <part name="P+3" library="supply1" library_urn="urn:adsk.eagle:library:371" deviceset="VCC" device=""/>
 <part name="CHARGER" library="B2B-XH-A" deviceset="B2B-XH-A" device=""/>
-<part name="P+4" library="supply1" library_urn="urn:adsk.eagle:library:371" deviceset="VCC" device=""/>
 <part name="JP1" library="pinhead" library_urn="urn:adsk.eagle:library:325" deviceset="PINHD-1X2" device="" package3d_urn="urn:adsk.eagle:package:22435/2"/>
 <part name="C3" library="CL31B106KAHNNNE" deviceset="CL31B106KAHNNNE" device=""/>
 <part name="C1" library="CL31B106KAHNNNE" deviceset="CL31B106KAHNNNE" device=""/>
 <part name="U1" library="HT7333" deviceset="HT7333" device=""/>
-<part name="LED1" library="led" library_urn="urn:adsk.eagle:library:259" deviceset="TLLR4400" device="" package3d_urn="urn:adsk.eagle:package:15797/1"/>
+<part name="LED1" library="led" deviceset="TLLR4400" device="" package3d_urn="urn:adsk.eagle:package:15797/1"/>
 <part name="P+5" library="supply1" library_urn="urn:adsk.eagle:library:371" deviceset="VCC" device=""/>
 <part name="P+6" library="supply1" library_urn="urn:adsk.eagle:library:371" deviceset="VCC" device=""/>
@@
 <attribute name="NAME" x="-17.78" y="95.25" size="1.778" layer="95" rot="R180"/>
 <attribute name="VALUE" x="-17.78" y="106.68" size="1.778" layer="96" rot="R180"/>
-</instance>
-<instance part="P+4" gate="VCC" x="86.36" y="43.18" smashed="yes">
-<attribute name="VALUE" x="83.82" y="40.64" size="1.778" layer="96" rot="R90"/>
 </instance>
 <instance part="JP1" gate="G$1" x="5.08" y="99.06" smashed="yes">
@@
 </segment>
 <segment>
-<pinref part="U2" gate="G$1" pin="ADO"/>
-<wire x1="96.52" y1="38.1" x2="86.36" y2="38.1" width="0.1524" layer="91"/>
-<pinref part="P+4" gate="VCC" pin="VCC"/>
-<wire x1="86.36" y1="38.1" x2="86.36" y2="40.64" width="0.1524" layer="91"/>
-</segment>
-<segment>
